File: hardware/relay_circuit.sch (KiCad schematic (older format))
At the start: 4 parts

Commit message: layout first draft
Parts:
- R33: renamed from R?; footprint (none) -> Resistor_SMD:R_0805_2012Metric_Pad1.15x1.40mm_HandSolder
- gave numbers to parts that had none: 3
Connections:
- net LINE: now also K6.2; no longer K6.3
- net line_switched: now also K6.3; no longer K6.2
Changed lines of the file:
@@
 $Descr A4 11693 8268
 encoding utf-8
-Sheet 10 10
+Sheet 7 10
 Title ""
 Date ""
@@
 P 3350 2900
 AR Path="/5C0C8264" Ref="K?"  Part="1"
-AR Path="/5C0C80CB/5C0C8264" Ref="K?"  Part="1"
-AR Path="/5C0C995E/5C0C8264" Ref="K?"  Part="1"
-AR Path="/5C0C99E3/5C0C8264" Ref="K?"  Part="1"
-AR Path="/5C0C9B56/5C0C8264" Ref="K?"  Part="1"
-AR Path="/5C0C9BDB/5C0C8264" Ref="K?"  Part="1"
-AR Path="/5C14D74F/5C0C8264" Ref="K?"  Part="1"
-F 0 "K?" H 3780 2946 50  0000 L CNN
+AR Path="/5C0C80CB/5C0C8264" Ref="K6"  Part="1"
+AR Path="/5C0C995E/5C0C8264" Ref="K5"  Part="1"
+AR Path="/5C0C99E3/5C0C8264" Ref="K4"  Part="1"
+AR Path="/5C0C9B56/5C0C8264" Ref="K3"  Part="1"
+AR Path="/5C0C9BDB/5C0C8264" Ref="K2"  Part="1"
+AR Path="/5C14D74F/5C0C8264" Ref="K1"  Part="1"
+F 0 "K6" H 3780 2946 50  0000 L CNN
 F 1 "G5Q-1" H 3780 2855 50  0000 L CNN
 F 2 "Relay_THT:Relay_SPDT_Omron-G5Q-1" H 3800 2850 50  0001 L CNN
@@
 $EndComp
 $Comp
-L power:+5V #PWR0113
+L power:+5V #PWR087
 U 1 1 5C0C8291
 P 3150 2600
-AR Path="/5C0C80CB/5C0C8291" Ref="#PWR0113"  Part="1"
-AR Path="/5C0C995E/5C0C8291" Ref="#PWR?"  Part="1"
-AR Path="/5C0C99E3/5C0C8291" Ref="#PWR?"  Part="1"
-AR Path="/5C0C9B56/5C0C8291" Ref="#PWR?"  Part="1"
-AR Path="/5C0C9BDB/5C0C8291" Ref="#PWR?"  Part="1"
-AR Path="/5C14D74F/5C0C8291" Ref="#PWR?"  Part="1"
-F 0 "#PWR?" H 3150 2450 50  0001 C CNN
+AR Path="/5C0C80CB/5C0C8291" Ref="#PWR087"  Part="1"
+AR Path="/5C0C995E/5C0C8291" Ref="#PWR084"  Part="1"
+AR Path="/5C0C99E3/5C0C8291" Ref="#PWR081"  Part="1"
+AR Path="/5C0C9B56/5C0C8291" Ref="#PWR078"  Part="1"
+AR Path="/5C0C9BDB/5C0C8291" Ref="#PWR075"  Part="1"
+AR Path="/5C14D74F/5C0C8291" Ref="#PWR072"  Part="1"
+F 0 "#PWR087" H 3150 2450 50  0001 C CNN
 F 1 "+5V" H 3165 2773 50  0000 C CNN
 F 2 "" H 3150 2600 50  0001 C CNN
@@
 $EndComp
 $Comp
-L Transistor_FET:2N7002 Q?
+L Transistor_FET:2N7002 Q10
 U 1 1 5C0C82C4
 P 3050 3650
-AR Path="/5C0C80CB/5C0C82C4" Ref="Q?"  Part="1"
-AR Path="/5C0C995E/5C0C82C4" Ref="Q?"  Part="1"
-AR Path="/5C0C99E3/5C0C82C4" Ref="Q?"  Part="1"
-AR Path="/5C0C9B56/5C0C82C4" Ref="Q?"  Part="1"
-AR Path="/5C0C9BDB/5C0C82C4" Ref="Q?"  Part="1"
-AR Path="/5C14D74F/5C0C82C4" Ref="Q?"  Part="1"
-F 0 "Q?" V 3300 3700 50  0000 L CNN
+AR Path="/5C0C80CB/5C0C82C4" Ref="Q10"  Part="1"
+AR Path="/5C0C995E/5C0C82C4" Ref="Q9"  Part="1"
+AR Path="/5C0C99E3/5C0C82C4" Ref="Q8"  Part="1"
+AR Path="/5C0C9B56/5C0C82C4" Ref="Q7"  Part="1"
+AR Path="/5C0C9BDB/5C0C82C4" Ref="Q6"  Part="1"
+AR Path="/5C14D74F/5C0C82C4" Ref="Q5"  Part="1"
+F 0 "Q10" V 3300 3700 50  0000 L CNN
 F 1 "2N7002" V 3300 3300 50  0000 L CNN
 F 2 "Package_TO_SOT_SMD:SOT-23" H 3250 3575 50  0001 L CIN
@@
 P 3150 3850
 AR Path="/5C0C85D6" Ref="#PWR?"  Part="1"
-AR Path="/5C0C80CB/5C0C85D6" Ref="#PWR0114"  Part="1"
-AR Path="/5C0C995E/5C0C85D6" Ref="#PWR?"  Part="1"
-AR Path="/5C0C99E3/5C0C85D6" Ref="#PWR?"  Part="1"
-AR Path="/5C0C9B56/5C0C85D6" Ref="#PWR?"  Part="1"
-AR Path="/5C0C9BDB/5C0C85D6" Ref="#PWR?"  Part="1"
-AR Path="/5C14D74F/5C0C85D6" Ref="#PWR?"  Part="1"
-F 0 "#PWR?" H 3150 3600 50  0001 C CNN
+AR Path="/5C0C80CB/5C0C85D6" Ref="#PWR088"  Part="1"
+AR Path="/5C0C995E/5C0C85D6" Ref="#PWR085"  Part="1"
+AR Path="/5C0C99E3/5C0C85D6" Ref="#PWR082"  Part="1"
+AR Path="/5C0C9B56/5C0C85D6" Ref="#PWR079"  Part="1"
+AR Path="/5C0C9BDB/5C0C85D6" Ref="#PWR076"  Part="1"
+AR Path="/5C14D74F/5C0C85D6" Ref="#PWR073"  Part="1"
+F 0 "#PWR088" H 3150 3600 50  0001 C CNN
 F 1 "GND" H 3150 3700 50  0000 C CNN
 F 2 "" H 3150 3850 50  0000 C CNN
@@
 $EndComp
 $Comp
-L Device:R R?
+L Device:R R33
 U 1 1 5C0C8788
 P 2700 3650
-AR Path="/5C0C80CB/5C0C8788" Ref="R?"  Part="1"
-AR Path="/5C0C995E/5C0C8788" Ref="R?"  Part="1"
-AR Path="/5C0C99E3/5C0C8788" Ref="R?"  Part="1"
-AR Path="/5C0C9B56/5C0C8788" Ref="R?"  Part="1"
-AR Path="/5C0C9BDB/5C0C8788" Ref="R?"  Part="1"
-AR Path="/5C14D74F/5C0C8788" Ref="R?"  Part="1"
-F 0 "R?" V 2493 3650 50  0000 C CNN
+AR Path="/5C0C80CB/5C0C8788" Ref="R33"  Part="1"
+AR Path="/5C0C995E/5C0C8788" Ref="R32"  Part="1"
+AR Path="/5C0C99E3/5C0C8788" Ref="R31"  Part="1"
+AR Path="/5C0C9B56/5C0C8788" Ref="R30"  Part="1"
+AR Path="/5C0C9BDB/5C0C8788" Ref="R29"  Part="1"
+AR Path="/5C14D74F/5C0C8788" Ref="R28"  Part="1"
+F 0 "R33" V 2493 3650 50  0000 C CNN
 F 1 "100R" V 2584 3650 50  0000 C CNN
-F 2 "" V 2630 3650 50  0001 C CNN
+F 2 "Resistor_SMD:R_0805_2012Metric_Pad1.15x1.40mm_HandSolder" V 2630 3650 50  0001 C CNN
 F 3 "~" H 2700 3650 50  0001 C CNN
 	1    2700 3650
@@
 gate
 $Comp
-L Diode:BAT54A D?
+L Diode:BAT54A D6
 U 1 1 5C0C8CF6
 P 2450 2900
-AR Path="/5C0C80CB/5C0C8CF6" Ref="D?"  Part="1"
-AR Path="/5C0C995E/5C0C8CF6" Ref="D?"  Part="1"
-AR Path="/5C0C99E3/5C0C8CF6" Ref="D?"  Part="1"
-AR Path="/5C0C9B56/5C0C8CF6" Ref="D?"  Part="1"
-AR Path="/5C0C9BDB/5C0C8CF6" Ref="D?"  Part="1"
-AR Path="/5C14D74F/5C0C8CF6" Ref="D?"  Part="1"
-F 0 "D?" V 2404 2988 50  0000 L CNN
+AR Path="/5C0C80CB/5C0C8CF6" Ref="D6"  Part="1"
+AR Path="/5C0C995E/5C0C8CF6" Ref="D5"  Part="1"
+AR Path="/5C0C99E3/5C0C8CF6" Ref="D4"  Part="1"
+AR Path="/5C0C9B56/5C0C8CF6" Ref="D3"  Part="1"
+AR Path="/5C0C9BDB/5C0C8CF6" Ref="D2"  Part="1"
+AR Path="/5C14D74F/5C0C8CF6" Ref="D1"  Part="1"
+F 0 "D6" V 2404 2988 50  0000 L CNN
 F 1 "BAT54A" V 2495 2988 50  0000 L CNN
 F 2 "Package_TO_SOT_SMD:SOT-23" H 2525 3025 50  0001 L CNN
@@
 Connection ~ 3150 3200
 $Comp
-L power:LINE #PWR?
+L power:LINE #PWR089
 U 1 1 5C0C934A
-P 3650 2600
-AR Path="/5C0C80CB/5C0C934A" Ref="#PWR?"  Part="1"
-AR Path="/5C0C995E/5C0C934A" Ref="#PWR?"  Part="1"
-AR Path="/5C0C99E3/5C0C934A" Ref="#PWR?"  Part="1"
-AR Path="/5C0C9B56/5C0C934A" Ref="#PWR?"  Part="1"
-AR Path="/5C0C9BDB/5C0C934A" Ref="#PWR?"  Part="1"
-AR Path="/5C14D74F/5C0C934A" Ref="#PWR?"  Part="1"
-F 0 "#PWR?" H 3650 2450 50  0001 C CNN
-F 1 "LINE" H 3667 2773 50  0000 C CNN
-F 2 "" H 3650 2600 50  0001 C CNN
-F 3 "" H 3650 2600 50  0001 C CNN
-	1    3650 2600
-	1    0    0    -1
+P 3550 3200
+AR Path="/5C0C80CB/5C0C934A" Ref="#PWR089"  Part="1"
+AR Path="/5C0C995E/5C0C934A" Ref="#PWR086"  Part="1"
+AR Path="/5C0C99E3/5C0C934A" Ref="#PWR083"  Part="1"
+AR Path="/5C0C9B56/5C0C934A" Ref="#PWR080"  Part="1"
+AR Path="/5C0C9BDB/5C0C934A" Ref="#PWR077"  Part="1"
+AR Path="/5C14D74F/5C0C934A" Ref="#PWR074"  Part="1"
+F 0 "#PWR089" H 3550 3050 50  0001 C CNN
+F 1 "LINE" H 3567 3373 50  0000 C CNN
+F 2 "" H 3550 3200 50  0001 C CNN
+F 3 "" H 3550 3200 50  0001 C CNN
+	1    3550 3200
+	-1   0    0    1
 $EndComp
-Text HLabel 3550 3200 3    50   Output ~ 0
+Text HLabel 3650 2600 1    50   Output ~ 0
 line_switched
 $EndSCHEMATC
